File: bts7960 adapter/bts7960 adapter.kicad_sch (KiCad schematic)
At the start: 7 parts, among them J1 Conn_01x05, J2 Conn_02x04_Odd_Even, Q1 AO3400A, Q2 AO3400A

Commit message: done
Parts:
- J1: footprint Connector_PinHeader_2.54mm:PinHeader_1x05_P2.54mm_Vertical -> 1KicadLib:1x05_wire2board
Changed lines of the file:
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@@
 			)
 		)
-		(property "Footprint" "Connector_PinHeader_2.54mm:PinHeader_1x05_P2.54mm_Vertical"
+		(property "Footprint" "1KicadLib:1x05_wire2board"
 			(at 26.035 97.79 0)
 			(effects
